Commit message: Full Refactoring and code cleanup

File: src/omni_base/urdf/omniserv.urdf (robot description, URDF)
Before this commit: robot omniserv, 10 links, 9 joints
Links:
- added link ir_back; visual box size=0.02 0.02 0.02
- added link ir_front; visual box size=0.02 0.02 0.02
- added link ir_left; visual box size=0.02 0.02 0.02
- added link ir_right; visual box size=0.02 0.02 0.02
- added link us_front_center; visual box size=0.02 0.04 0.02
- added link us_front_left; visual box size=0.02 0.04 0.02
- added link us_front_right; visual box size=0.02 0.04 0.02
- added link us_rear_center; visual box size=0.02 0.04 0.02
- added link us_rear_left; visual box size=0.02 0.04 0.02
- added link us_rear_right; visual box size=0.02 0.04 0.02
Joints:
- added joint base_to_ir_back: type fixed, parent base_link, child ir_back, origin xyz=-0.32 0.0 0.05 rpy=0 1.5708 0
- added joint base_to_ir_front: type fixed, parent base_link, child ir_front, origin xyz=0.32 0.0 0.05 rpy=0 1.5708 0
- added joint base_to_ir_left: type fixed, parent base_link, child ir_left, origin xyz=0.0 0.32 0.05 rpy=0 1.5708 0
- added joint base_to_ir_right: type fixed, parent base_link, child ir_right, origin xyz=0.0 -0.32 0.05 rpy=0 1.5708 0
- added joint base_to_us_front_center: type fixed, parent base_link, child us_front_center, origin xyz=0.30 0.0 0.05 rpy=0 0 0
- added joint base_to_us_front_left: type fixed, parent base_link, child us_front_left, origin xyz=0.26 0.15 0.05 rpy=0 0 0.6
- added joint base_to_us_front_right: type fixed, parent base_link, child us_front_right, origin xyz=0.26 -0.15 0.05 rpy=0 0 -0.6
- added joint base_to_us_rear_center: type fixed, parent base_link, child us_rear_center, origin xyz=-0.30 0.0 0.05 rpy=0 0 3.14159
- added joint base_to_us_rear_left: type fixed, parent base_link, child us_rear_left, origin xyz=-0.26 0.15 0.05 rpy=0 0 2.54159
- added joint base_to_us_rear_right: type fixed, parent base_link, child us_rear_right, origin xyz=-0.26 -0.15 0.05 rpy=0 0 3.74159
